Commit message: full control

File: drone.urdf (robot description, URDF)
Before this commit: robot simple_drone, 4 links, 3 joints
Links:
- link nose_link: geometry visual box size=0.05 0.05 0.001
- link tail_link: geometry visual box size=0.05 0.05 0.001
Joints:
- joint base_to_nose: origin xyz=0.1 0 0.02 rpy=0 0 0 -> xyz=0.04 0 0.01 rpy=0 0 0
- joint base_to_tail: origin xyz=-0.1 0 0.02 rpy=0 0 0 -> xyz=-0.04 0 0.01 rpy=0 0 0
